Commit message: add dof

File: assets/urdf/centauro_urdf/urdf/centauro_sliding.urdf (robot description, URDF)
Before this commit: robot centauro, 27 links, 26 joints
Links:
- removed link D435_head_camera_bottom_screw_frame
- removed link D435_head_camera_link
- removed link D435i_camera_bottom_screw_frame
- removed link D435i_camera_link
Joints:
- removed joint D435_head_camera_joint
- removed joint D435_head_camera_link_joint
- removed joint D435i_camera_joint
- removed joint D435i_camera_link_joint
- removed joint d435_head_joint
- removed joint neck_base
- removed joint velodyne_joint

Commit message: limit pelvis rotation

File: assets/urdf/centauro_urdf/urdf/centauro_sliding.urdf (robot description, URDF)
Before this commit: robot centauro, 23 links, 19 joints
Joints:
- joint torso_yaw: limit lower=-2.618 upper=2.618 effort=147 velocity=5.7 -> lower=-0.5 upper=0.5 effort=147 velocity=5.7
- joint x_slider: limit lower=-5 upper=5 effort=100 velocity=1 -> lower=-0.5 upper=0.5 effort=100 velocity=1
- joint y_slider: limit lower=-5 upper=5 effort=100 velocity=1 -> lower=-0.5 upper=0.5 effort=100 velocity=1
- joint z_slider: limit lower=0 upper=1 effort=100 velocity=1 -> lower=0 upper=0.5 effort=100 velocity=1

Commit message: update CentauroPick

File: assets/urdf/centauro_urdf/urdf/centauro_sliding.urdf (robot description, URDF)
Before this commit: robot centauro, 23 links, 19 joints
Joints:
- joint pelvis_pitch_joint: limit lower=-1.57 upper=1.57 effort=0 velocity=0.5 -> lower=-0.2 upper=0.2 effort=0 velocity=0.5
- joint pelvis_roll_joint: limit lower=-1.57 upper=1.57 effort=0 velocity=0.5 -> lower=-0.2 upper=0.2 effort=0 velocity=0.5
