Commit message: update centauro cabinet training

File: assets/urdf/centauro_urdf/urdf/centauro_sliding_upperbody.urdf (robot description, URDF)
Before this commit: robot centauro, 36 links, 35 joints
Links:
- link pelvis: mass 1800.845851 -> 180.845851
Joints:
- joint pelvis_pitch_joint: limit lower=-0.2 upper=0.2 effort=10000 velocity=0.5 -> lower=-0.1 upper=0.1 effort=10000 velocity=0.5
- joint pelvis_roll_joint: limit lower=-0.2 upper=0.2 effort=10000 velocity=0.5 -> lower=-0.1 upper=0.1 effort=10000 velocity=0.5
- joint x_slider: limit lower=-0.5 upper=0.5 effort=10000 velocity=1 -> lower=-0.5 upper=0.1 effort=10000 velocity=1
- joint z_slider: limit lower=0 upper=0.5 effort=10000 velocity=1 -> lower=0 upper=1.0 effort=10000 velocity=1
