Commit message: add env CentauroDoor

File: assets/urdf/door.urdf (robot description, URDF)
Before this commit: robot urdf_door, 3 links, 2 joints
Links:
- removed link baseLink
- removed link childA
- removed link world
- added link door_handle, mass 0.1; collision box size=0.02 0.1 0.02; visual box size=0.02 0.1 0.02
- added link door_panel, mass 10; collision box size=0.05 0.8 2.0; visual box size=0.05 0.8 2.0
- added link hinge_post; collision cylinder length=2.0 radius=0.05; visual cylinder length=2.0 radius=0.05
Joints:
- removed joint fixed
- removed joint joint_baseLink_childA
- added joint door_hinge: type revolute, parent hinge_post, child door_panel, origin xyz=0 0 0.0, axis 0 0 1, limit lower=0.0 upper=1.57 effort=10.0 velocity=1.0
- added joint handle_hinge: type revolute, parent door_panel, child door_handle, origin xyz=0.026 0.78 0.1, axis 1 0 0, limit lower=0.0 upper=0.5 effort=10.0 velocity=1.0

Commit message: fix door

File: assets/urdf/door.urdf (robot description, URDF)
Before this commit: robot simple_door_with_handle, 3 links, 2 joints
Joints:
- joint door_hinge: limit lower=0.0 upper=1.57 effort=10.0 velocity=1.0 -> lower=0.0 upper=0.0 effort=10.0 velocity=1.0
