Commit message: door left

File: assets/urdf/door_left.urdf (robot description, URDF)
Before this commit: robot simple_door_with_handle, 3 links, 2 joints
Joints:
- joint door_hinge: limit lower=0.0 upper=0.0 effort=10.0 velocity=1.0 -> lower=0.0 upper=0.0001 effort=10.0 velocity=1.0
- joint handle_hinge: limit lower=0.0 upper=-0.5 effort=10.0 velocity=1.0 -> lower=-0.5 upper=0.0 effort=10.0 velocity=1.0; origin xyz=0.026 0.78 0.1 -> xyz=0.026 -0.78 0.1
