Commit message: centauro dual arm

File: assets/urdf/dual_box.urdf (robot description, URDF)
Before this commit: robot box_with_plate, 2 links, 1 joints
Links:
- link box: geometry collision box size=0.3 0.3 0.2; visual box size=0.2 0.2 0.2
- link plate: geometry collision box size=0.3 0.3 0.1; visual box size=0.4 0.4 0.1
